Commit message: Change camera pose for better view

File: urdf/my_model.xacro (robot description, xacro)
@@ -133,5 +133,5 @@
   <xacro:macro name="camera_link" params="parent">
     <link name="camera_link">
-	<origin xyz="${0} ${0} ${camera_z}" rpy="0 0 0" />
+	<origin xyz="${left2_wheel_x} ${left2_wheel_y} ${camera_z}" rpy="0 0 ${M_PI/2 + M_PI/6}" />
       <collision>
         <geometry>
@@ -152,5 +152,5 @@
         <parent link="${parent}"/>
         <child link="camera_link"/>
-        <origin xyz="${0} ${0} ${camera_z}" rpy="0 0 0" />
+        <origin xyz="${left2_wheel_x} ${left2_wheel_y} ${camera_z}" rpy="0 0 ${M_PI/2 + M_PI/6}" />
         <axis xyz="1 0 0" />
     </joint>
